Commit message: courier com 1 metro e caixas nas lateriais

File: src/courier_description/urdf/robot.urdf (robot description, URDF)
Before this commit: robot courier, 10 links, 9 joints
Links:
- removed link ultrasson
- added link compartimento2; collision box size=0.3 0.3 0.1; visual box size=0.3 0.3 0.1
- added link compartimento3; collision box size=0.3 0.3 0.1; visual box size=0.3 0.3 0.1
- added link compartimento4; collision box size=0.3 0.3 0.1; visual box size=0.3 0.3 0.1
- added link compartimento5; collision box size=0.3 0.3 0.1; visual box size=0.3 0.3 0.1
- added link tampa_compartimento2; visual box size=0.3 0.01 0.1
- added link tampa_compartimento3; visual box size=0.3 0.01 0.1
- added link tampa_compartimento4; visual box size=0.3 0.01 0.1
- added link tampa_compartimento5; visual box size=0.3 0.01 0.1
- link base: geometry visual box size=0.4 0.4 1
- link espaco_camera: geometry visual box size=0.01 0.35 0.15
- link tampa_compartimento: geometry visual box size=0.3 0.01 0.1
Joints:
- removed joint base_to_ultrasson
- added joint base_to_compartimento2: type fixed, parent base, child compartimento2, origin xyz=0 0 0.20 rpy=0 0 0
- added joint base_to_compartimento3: type fixed, parent base, child compartimento3, origin xyz=0 0 0.40 rpy=0 0 0
- added joint base_to_compartimento4: type fixed, parent base, child compartimento4, origin xyz=0 0 -0.20 rpy=0 0 0
- added joint base_to_compartimento5: type fixed, parent base, child compartimento5, origin xyz=0 0 -0.40 rpy=0 0 0
- added joint base_to_tampa2: type fixed, parent compartimento, child tampa_compartimento2, origin xyz=0 0.21 0.20 rpy=0 0 0
- added joint base_to_tampa3: type fixed, parent compartimento, child tampa_compartimento3, origin xyz=0 0.21 0.40 rpy=0 0 0
- added joint base_to_tampa4: type fixed, parent compartimento, child tampa_compartimento4, origin xyz=0 0.21 -0.20 rpy=0 0 0
- added joint base_to_tampa5: type fixed, parent compartimento, child tampa_compartimento5, origin xyz=0 0.21 -0.40 rpy=0 0 0
- joint base_to_compartimento: origin xyz=0 0 0.05 rpy=0 0 0 -> xyz=0 0 0.0 rpy=0 0 0
- joint base_to_espaco_camera: origin xyz=0.18 0.0 0.05 rpy=0 0 0 -> xyz=0.2 0.0 0.35 rpy=0 0 0
- joint base_to_lidar: origin xyz=0.176 0 0.11 rpy=0 0 0 -> xyz=0.176 0 0.51 rpy=0 0 0
- joint base_to_roda1: origin xyz=0.2 0.2 -0.1 rpy=1.5708 0 0 -> xyz=0.2 0.2 -0.5 rpy=1.5708 0 0
- joint base_to_roda2: origin xyz=0.2 -0.2 -0.1 rpy=1.5708 0 0 -> xyz=0.2 -0.2 -0.5 rpy=1.5708 0 0
- joint base_to_roda3: origin xyz=-0.2 -0.2 -0.1 rpy=1.5708 0 0 -> xyz=-0.2 -0.2 -0.5 rpy=1.5708 0 0
- joint base_to_roda4: origin xyz=-0.2 0.2 -0.1 rpy=1.5708 0 0 -> xyz=-0.2 0.2 -0.5 rpy=1.5708 0 0
- joint base_to_tampa: origin xyz=0 0 0.05 rpy=0 0 0 -> xyz=0 0.21 0.0 rpy=0 0 0
